Commit message: Added demo worlds

File: src/gz_spray_painting_plugin_demo/urdf/spray_nozzle.urdf (robot description, URDF)
Before this commit: robot spray_gun_robot, 2 links, 1 joints
Links:
- link spray_gun_base_link: geometry visual mesh filename=package://gz_spray_painting_plugin_demo/meshes/spray_gun/sp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 scale=1 1 1
Joints:
- joint nozzle_joint: origin xyz=0.12 0 0.1 rpy=0 -0.25 0 -> xyz=0.0 -0.13 0.16 rpy=0.0 -1.57 0.0

File: src/gz_spray_painting_plugin_demo/urdf/ur_spray_gz.urdf.xacro (robot description, xacro)
@@ -133,5 +133,5 @@
       <origin xyz="0 0 0" rpy="0 0 0"/>
       <geometry>
-        <mesh filename="package://gz_sim_spray_painting_plugin/meshes/spray_gun/spray_gun.glb" scale="1 1 1"/>
+        <mesh filename="package://gz_spray_painting_plugin_demo/meshes/spray_gun/spray_gun.glb" scale="1 1 1"/>
       </geometry>
     </visual>
